File: Hardware/SparkFun_AS7343_Qwiic.kicad_pcb (KiCad board)
At the start: 2 copper layers, 25.4 x 25.4 mm, 64 parts, among them J1 Qwiic_RA, J2 Qwiic_RA, J3 Conn_01x06, Q1 BSS138, Q2 BSS138, U1 RT9080-1.8V, U2 AS7343

Commit message: fixed logic level converters
-body diodes in LLC transistors were allowing high side voltage into low side. (This was incorrect in v01).
-fixed LLC circuit to have low/high voltages on the correct sides
-rerouted
-bumped version to v02
Parts:
- turned Q1 to 180 degrees
- turned Q2 to 180 degrees
Connections:
- Q1 pad 1: 3.3V -> 1.8V
- Q1 pad 2: SCL -> SCL_1V8
- Q1 pad 3: SCL_1V8 -> SCL
- Q2 pad 1: 3.3V -> 1.8V
- Q2 pad 2: SDA -> SDA_1V8
- Q2 pad 3: SDA_1V8 -> SDA
Routing:
- net 3.3V: track 74.7 -> 65.4 mm, vias 8 -> 7
- net 1.8V: track 27.4 -> 30.6 mm
- net Net-(JP2-A): track 3.49 -> 5.30 mm
- net SCL: track 49.1 -> 50.7 mm
- net SDA_1V8: track 15.9 -> 16.5 mm
- net GND: vias 55 -> 56
Other:
- board text added: "v02"
- board text removed: "v01"

Commit message: bumped version to v10 in sch and pcb
Other:
- board text added: "v10"
- board text removed: "v02"
Changed lines of the file:
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@@
 	(title_block
 		(title "SparkFun Spectral Sensor Breakout AS7353 Qwiic")
-		(date "2025-04-22")
-		(rev "v02")
+		(date "2025-05-05")
+		(rev "v10")
 		(company "SparkFun Electronics")
 		(comment 1 "Based off the AS726X Qwiic by N. Seidle")
@@
 		(layer "Edge.Cuts")
 	)
-	(gr_text "v02"
+	(gr_text "v10"
 		(at 124.192 98.263 270)
 		(layer "B.Cu" knockout)

Commit message: eng checklist run for v10
-updated soldermask color to red
-library update on the DNP 5mm pth LED (linking due to new naming)
-library update on qwiic connector - looks like just an update on the courtyard
Parts:
- D3: footprint SparkFun-LED:LED_5MM -> SparkFun-LED:LED_5mm_PTH_Red_NoSilk
Other:
- board text added: "Solder Mask: Red"
- board text removed: "Solder Mask: Black"
